Commit message: code update

File: smart_factory/urdf/smart_factory.xacro (robot description, xacro)
@@ -79,5 +79,5 @@
     </visual>
     <!-- space limitation -->
-    <!-- table length: 1174mm, width: 620mm, height: 1100mm-->
+    <!-- table length: 1174mm, width: 630mm, height: 1100mm-->
     <collision>
       <origin rpy="0 0 0" xyz="0.287 0.22 0.55"/>
@@ -86,10 +86,10 @@
       </geometry>
     </collision>
-    <collision>
+    <!-- <collision>
       <origin rpy="0 0 0" xyz="0.287 -0.42 0.55"/>
       <geometry>
         <box size="1.174 0.01 1.1" />
       </geometry>
-    </collision>
+    </collision> -->
     <collision>
       <origin rpy="0 0 0" xyz="-0.3 -0.09 0.55"/>

Commit message: code update

File: smart_factory/urdf/smart_factory.xacro (robot description, xacro)
@@ -86,10 +86,10 @@
       </geometry>
     </collision>
-    <!-- <collision>
-      <origin rpy="0 0 0" xyz="0.287 -0.42 0.55"/>
+    <collision>
+      <origin rpy="0 0 0" xyz="0.287 -0.44 0.55"/>
       <geometry>
         <box size="1.174 0.01 1.1" />
       </geometry>
-    </collision> -->
+    </collision>
     <collision>
       <origin rpy="0 0 0" xyz="-0.3 -0.09 0.55"/>
